Commit message: Updating for fer vs fr3

File: franka_fer_moveit_config/srdf/fer_arm.srdf.xacro (robot description, xacro)
@@ -1,6 +1,6 @@
 <?xml version="1.0" ?>
-<robot xmlns:xacro="http://www.ros.org/wiki/xacro" name="fr3">
-  <xacro:macro name="fr3_arm" params="arm_id:='fr3' ">
-    <xacro:include filename="$(find franka_fr3_moveit_config)/srdf/group_definition.xacro"/>
+<robot xmlns:xacro="http://www.ros.org/wiki/xacro" name="fer">
+  <xacro:macro name="fer_arm" params="arm_id:='fer' ">
+    <xacro:include filename="$(find franka_fer_moveit_config)/srdf/group_definition.xacro"/>
     <xacro:group_definition arm_id="${arm_id}" group_name="${arm_id}_manipulator" tip_link="${arm_id}_hand_tcp"/>
     <xacro:group_definition arm_id="${arm_id}" group_name="${arm_id}_arm" tip_link="${arm_id}_link8"/>

File: franka_fer_moveit_config/srdf/group_definition.xacro (robot description, xacro)
@@ -1,4 +1,4 @@
 <?xml version="1.0" encoding="UTF-8"?>
-<robot xmlns:xacro="http://www.ros.org/wiki/xacro" name="fr3">
+<robot xmlns:xacro="http://www.ros.org/wiki/xacro" name="fer">
   <xacro:macro name="group_definition" params="group_name arm_id tip_link">
     <group name="${group_name}">

File: franka_fer_moveit_config/srdf/hand.xacro (robot description, xacro)
@@ -1,5 +1,5 @@
 <?xml version="1.0" ?>
-<robot xmlns:xacro="http://www.ros.org/wiki/xacro" name="fr3">
-  <xacro:macro name="hand" params="arm_id:='fr3' ">
+<robot xmlns:xacro="http://www.ros.org/wiki/xacro" name="fer">
+  <xacro:macro name="hand" params="arm_id:='fer' ">
     <group name="hand">
       <link name="${arm_id}_hand"/>
